Commit message: Add files via upload

File: catkin_ws/src/my_robot/urdf/my_robot.xacro (robot description, xacro)
@@ -28,5 +28,5 @@
 		<geometry>
 			<box size=".4 .2 .1"/>
-		</geoetry>
+		</geometry>
 	</visual>
 	<collision name='back_caster_collision'>

Commit message: Update my_robot.xacro

File: catkin_ws/src/my_robot/urdf/my_robot.xacro (robot description, xacro)
@@ -106,8 +106,8 @@
   </gazebo>
   <gazebo reference="right_wheel">
-    <material>Gazebo/Red</material>
+    <material>Gazebo/Blue</material>
   </gazebo>
   <joint type="continuous" name="left_wheel_hinge">
-    <origin xyz="0 0.325 0" rpy="0 0 0" />
+    <origin xyz="0 0.15 0" rpy="0 0 0" />
     <child link="left_wheel" />
     <parent link="chassis" />
@@ -117,5 +117,5 @@
   </joint>
   <joint type="continuous" name="right_wheel_hinge">
-    <origin xyz="0 -0.325 0" rpy="0 0 0" />
+    <origin xyz="0 -0.15 0" rpy="0 0 0" />
     <child link="right_wheel" />
     <parent link="chassis" />
@@ -143,5 +143,5 @@
   </gazebo>
   <joint type="fixed" name="camera_joint">
-    <origin xyz="0.3 0 0" rpy="0 0 0" />
+    <origin xyz="0.2 0 0" rpy="0 0 0" />
     <parent link="chassis" />
     <child link="camera" />
@@ -175,3 +175,2 @@
   </joint>
 </robot>
-</robot>

Commit message: Update my_robot.xacro

File: catkin_ws/src/my_robot/urdf/my_robot.xacro (robot description, xacro)
@@ -170,5 +170,5 @@
   </link>
   <joint name="hokuyo" type="fixed">
-    <origin xyz="0.25 0 0.08" rpy="0 0 0"/>
+    <origin xyz="0.15 0 0.1" rpy="0 0 0"/>
     <parent link="chassis" />
     <child link="hokuyo" />
